File: mux-control.sch (KiCad schematic (older format))
At the start: 14 parts, among them J1 Conn_01x08, SW1 SW_Push_Dual, SW2 SW_Push_Dual, SW3 SW_Push_Dual, SW4 SW_Push_Dual, U1 CD74HC4051E

Commit message: new design
Parts:
- D1: footprint LED_THT:LED_D4.0mm -> Resistor_THT:R_Axial_DIN0204_L3.6mm_D1.6mm_P2.54mm_Vertical
- J1: footprint Connector_PinHeader_2.00mm:PinHeader_1x08_P2.00mm_Vertical -> Connector_PinHeader_1.00mm:PinHeader_1x08_P1.00mm_Horizontal
- U1: symbol mux-control-rescue:CD74HC4051E-CD74HC4051E -> CD74HC4051E:CD74HC4051E
Changed lines of the file:
@@
 F 0 "J1" H 8080 1792 50  0000 L CNN
 F 1 "Conn_01x08" H 8080 1701 50  0000 L CNN
-F 2 "Connector_PinHeader_2.00mm:PinHeader_1x08_P2.00mm_Vertical" H 8000 1800 50  0001 C CNN
+F 2 "Connector_PinHeader_1.00mm:PinHeader_1x08_P1.00mm_Horizontal" H 8000 1800 50  0001 C CNN
 F 3 "~" H 8000 1800 50  0001 C CNN
 	1    8000 1800
@@
 F 0 "D1" H 4343 3867 50  0000 C CNN
 F 1 "LED" H 4343 3776 50  0000 C CNN
-F 2 "LED_THT:LED_D4.0mm" H 4350 3650 50  0001 C CNN
+F 2 "Resistor_THT:R_Axial_DIN0204_L3.6mm_D1.6mm_P2.54mm_Vertical" H 4350 3650 50  0001 C CNN
 F 3 "~" H 4350 3650 50  0001 C CNN
 	1    4350 3650
@@
 	3700 2100 3700 1500
 $Comp
-L mux-control-rescue:CD74HC4051E-CD74HC4051E U1
+L CD74HC4051E:CD74HC4051E U1
 U 1 1 5EF91C6E
 P 6000 2400

Commit message: autorouted
Parts:
- D1: footprint Resistor_THT:R_Axial_DIN0204_L3.6mm_D1.6mm_P2.54mm_Vertical -> LED_THT:LED_D4.0mm
- J1: footprint Connector_PinHeader_1.00mm:PinHeader_1x08_P1.00mm_Horizontal -> Connector_PinHeader_2.00mm:PinHeader_1x08_P2.00mm_Vertical
- U1: symbol CD74HC4051E:CD74HC4051E -> mux-control-rescue:CD74HC4051E-CD74HC4051E
Changed lines of the file:
@@
 F 0 "J1" H 8080 1792 50  0000 L CNN
 F 1 "Conn_01x08" H 8080 1701 50  0000 L CNN
-F 2 "Connector_PinHeader_1.00mm:PinHeader_1x08_P1.00mm_Horizontal" H 8000 1800 50  0001 C CNN
+F 2 "Connector_PinHeader_2.00mm:PinHeader_1x08_P2.00mm_Vertical" H 8000 1800 50  0001 C CNN
 F 3 "~" H 8000 1800 50  0001 C CNN
 	1    8000 1800
@@
 F 0 "D1" H 4343 3867 50  0000 C CNN
 F 1 "LED" H 4343 3776 50  0000 C CNN
-F 2 "Resistor_THT:R_Axial_DIN0204_L3.6mm_D1.6mm_P2.54mm_Vertical" H 4350 3650 50  0001 C CNN
+F 2 "LED_THT:LED_D4.0mm" H 4350 3650 50  0001 C CNN
 F 3 "~" H 4350 3650 50  0001 C CNN
 	1    4350 3650
@@
 	3700 2100 3700 1500
 $Comp
-L CD74HC4051E:CD74HC4051E U1
+L mux-control-rescue:CD74HC4051E-CD74HC4051E U1
 U 1 1 5EF91C6E
 P 6000 2400
